File: CW-PHONE-BAND-PASS/CW-PHONE-BAND-PASS.kicad_pcb (KiCad board)
At the start: 2 copper layers, 66 x 28 mm, 17 parts, among them J1 3F07_3.5mm, J2 3F07_3.5mm

Commit message: first PCB version released. Gerbers generated.
Parts:
- moved J1 0.50 mm to (106.5, 86.0)
- moved J2 0.50 mm to (159.5, 86.0)
Routing:
- net /OUT_R: track 6.35 -> 7.27 mm
- net /IN: track 35.4 -> 34.7 mm
Other:
- board text added: "20210823"
- board text added: "M210823A"
- board text removed: "20210820"

Commit message: pcb updated. gerber files rev 1 generated.
Parts:
- added G***: LOGO, pcblib_new599 Library:ARROW_6x4.5, F.Cu at (133.0, 76.5)
- added G***: LOGO, pcblib_new599 Library:ARROW_6x4.5, B.Cu at (113.0, 75.0)
- moved TP1 2.92 mm to (111.5, 78.5)
Routing:
- net /IN: track 34.7 -> 31.0 mm
- net /OUT_R: track 7.27 -> 6.56 mm
Other:
- outline, holes or cut-outs redrawn
- board text added: "20210901"
- board text added: "M210823A1"
- board text removed: "20210823"
- board text removed: "M210823A"
